File: schematic/v2.3/mMicroSD.brd (EAGLE design)
At the start: 38 x 18 mm, 23 parts, among them IC1 MAX3392, IC2 ATMEGA328, IC3 AD8531, J1 ISPTOUCH, M1 NTJD5121N

Commit message: Moved a few value labels around for better readability
Routing:
- net N$10: track 25.8 -> 27.7 mm
Changed lines of the file:
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@@
 <wire x1="38.000003125" y1="18.034" x2="0" y2="18.034" width="0.1778" layer="20"/>
 <wire x1="0" y1="18.034" x2="0" y2="0" width="0.1778" layer="20"/>
-<text x="2.11099375" y="8.983109375" size="1.016" layer="22" font="vector" rot="MR90">To M2/M4</text>
+<text x="2.11099375" y="9.364109375" size="1.016" layer="22" font="vector" rot="MR90">To M2/M4</text>
 <text x="33.98801875" y="8.094965625" size="1.016" layer="22" font="vector" rot="MR90">Extra mBus</text>
 <text x="28.362975" y="0.64" size="1.778" layer="21" font="vector" rot="R90">mMicroSD</text>
@@
 </element>
 <element name="R2" library="resistor" package="R0603" value="100k" x="2.0280875" y="6.38299375" smashed="yes" rot="MR90">
-<attribute name="VALUE" x="3.917021875" y="7.888746875" size="1.016" layer="22" font="vector" rot="MR0"/>
+<attribute name="VALUE" x="3.663021875" y="7.761746875" size="1.016" layer="22" font="vector" rot="MR0"/>
 </element>
 <element name="U$2" library="zz-kent" package="MBUS_IN" value="MBUS_IN" x="1.499996875" y="12.618975"/>
@@
 <element name="IC2" library="zz-kent" package="ATMEGA328" value="ATMEGA328" x="19.249925" y="8.11098125" smashed="yes" rot="MR0"/>
 <element name="IC1" library="haptics" package="14-TSSOP" value="MAX3392" x="6.999984375" y="4.61899375" smashed="yes" rot="MR90">
-<attribute name="VALUE" x="3.647184375" y="1.90119375" size="1.016" layer="22" font="vector" ratio="10" rot="MR180"/>
+<attribute name="VALUE" x="4.282184375" y="1.90119375" size="0.8128" layer="22" font="vector" ratio="10" rot="MR180"/>
 </element>
 <element name="R3" library="resistor" package="R0603" value="43k" x="24.39708125" y="14.812896875" smashed="yes" rot="MR270">
@@
 </element>
 <element name="IC3" library="haptics" package="SOT-23-5" value="AD8531" x="8.85393125" y="12.7039375" smashed="yes" rot="MR0">
-<attribute name="VALUE" x="12.02893125" y="9.9049375" size="1.016" layer="22" font="vector" ratio="10" rot="MR0"/>
+<attribute name="VALUE" x="11.13993125" y="10.1589375" size="0.8128" layer="22" font="vector" ratio="10" rot="MR0"/>
 </element>
 <element name="M1" library="haptics" package="SOT-363" value="NTJD5121N" x="27.7759125" y="10.4419375" smashed="yes" rot="MR0">
-<attribute name="VALUE" x="26.5899125" y="9.9009375" size="1.016" layer="22" font="vector" rot="MR0"/>
+<attribute name="VALUE" x="30.2729125" y="11.6789375" size="0.8128" layer="22" font="vector" rot="MR0"/>
 </element>
 <element name="R5" library="resistor" package="R0603" value="64k" x="14.0120375" y="15.8249625" smashed="yes" rot="MR270">
-<attribute name="VALUE" x="15.6630375" y="16.9679625" size="1.016" layer="22" font="vector" rot="MR270"/>
+<attribute name="VALUE" x="15.6630375" y="17.3489625" size="1.016" layer="22" font="vector" rot="MR270"/>
 </element>
 <element name="R7" library="resistor" package="R0603" value="33k" x="8.91196875" y="15.832959375" smashed="yes" rot="MR0">
@@
 <contactref element="R8" pad="1"/>
 <via x="29.21" y="10.541" extent="1-16" drill="0.3556"/>
-<wire x1="29.21" y1="10.541" x2="27.686" y2="8.636" width="0.1778" layer="1"/>
-<via x="27.686" y="8.636" extent="1-16" drill="0.3556"/>
-<wire x1="27.686" y1="8.636" x2="27.686" y2="9.552025" width="0.1778" layer="16"/>
+<wire x1="29.21" y1="10.541" x2="26.797" y2="10.541" width="0.1778" layer="1"/>
+<wire x1="26.797" y1="10.541" x2="26.416" y2="10.16" width="0.1778" layer="1"/>
+<wire x1="26.416" y1="10.16" x2="26.416" y2="8.636" width="0.1778" layer="1"/>
+<via x="26.416" y="8.636" extent="1-16" drill="0.3556"/>
+<wire x1="26.416" y1="8.636" x2="27.432" y2="8.636" width="0.1778" layer="16"/>
+<wire x1="27.432" y1="8.636" x2="27.686" y2="8.89" width="0.1778" layer="16"/>
+<wire x1="27.686" y1="8.89" x2="27.686" y2="9.552025" width="0.1778" layer="16"/>
 <wire x1="27.686" y1="9.552025" x2="27.7759125" y2="9.6419375" width="0.1778" layer="16"/>
 <wire x1="16.339925" y1="12.90348125" x2="16.339925" y2="10.711075" width="0.1778" layer="16"/>
@@
 <wire x1="25.273" y1="11.43" x2="25.273" y2="9.271" width="0.1778" layer="16"/>
 <wire x1="25.273" y1="9.271" x2="25.908" y2="8.636" width="0.1778" layer="16"/>
-<wire x1="25.908" y1="8.636" x2="27.686" y2="8.636" width="0.1778" layer="16"/>
+<wire x1="25.908" y1="8.636" x2="26.416" y2="8.636" width="0.1778" layer="16"/>
 <wire x1="29.21" y1="10.541" x2="29.21" y2="13.337909375" width="0.1778" layer="16"/>
 <wire x1="29.21" y1="13.337909375" x2="30.692103125" y2="14.6930125" width="0.1778" layer="16"/>
