File: schematic/v2.3/mMicroSD.brd (EAGLE design)
At the start: 38 x 18 mm, 23 parts, among them IC1 MAX3392, IC2 ATMEGA328, IC3 AD8531, J1 ISPTOUCH, M1 NTJD5121N

Commit message: Gave names to some previously anonymous lines
Connections:
- net N$11 renamed SD_CS
- net N$15 renamed SD_SCK
- net N$5 renamed SD_MISO
- net N$6 renamed SD_MOSI
Changed lines of the file:
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@@
 <wire x1="12.5840375" y1="14.9749625" x2="12.573" y2="14.986" width="0.1778" layer="16"/>
 </signal>
-<signal name="N$5">
+<signal name="SD_MISO">
 <contactref element="IC1" pad="5"/>
 <contactref element="SDCONN" pad="P$7"/>
@@
 <wire x1="3.890178125" y1="5.207" x2="4.082184375" y2="5.26899375" width="0.1778" layer="16"/>
 </signal>
-<signal name="N$6">
+<signal name="SD_MOSI">
 <contactref element="IC1" pad="4"/>
 <contactref element="SDCONN" pad="P$3"/>
@@
 <wire x1="4.035190625" y1="4.572" x2="4.082184375" y2="4.61899375" width="0.1778" layer="16"/>
 </signal>
-<signal name="N$11">
+<signal name="SD_CS">
 <contactref element="IC1" pad="3"/>
 <contactref element="SDCONN" pad="P$2"/>
@@
 <wire x1="4.050190625" y1="3.937" x2="4.082184375" y2="3.96899375" width="0.1778" layer="16"/>
 </signal>
-<signal name="N$15">
+<signal name="SD_SCK">
 <contactref element="IC1" pad="2"/>
 <contactref element="SDCONN" pad="P$5"/>
