File: schematic/v2.3/mMicroSD.sch (EAGLE design)
At the start: 23 parts, among them IC1 MAX3392, IC2 ATMEGA328, IC3 AD8531, J1 ISPTOUCH, M1 NTJD5121N

Commit message: Added some silkscreen to the board to make the orientation of two close resistors more apparent
Connections:
- net N$10 renamed GATE
- net N$17 renamed ADC_LINE
- net N$3 renamed DATA_LED
Changed lines of the file:
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@@
 </segment>
 </net>
-<net name="N$10" class="0">
+<net name="GATE" class="0">
 <segment>
 <pinref part="IC2" gate="G$1" pin="PC2"/>
@@
 </segment>
 </net>
-<net name="N$17" class="0">
+<net name="ADC_LINE" class="0">
 <segment>
 <pinref part="R3" gate="G$1" pin="1"/>
@@
 </segment>
 </net>
-<net name="N$3" class="0">
+<net name="DATA_LED" class="0">
 <segment>
 <pinref part="IC2" gate="G$1" pin="PC0"/>

Commit message: Gave names to some previously anonymous lines
Connections:
- net N$11 renamed SD_CS
- net N$15 renamed SD_SCK
- net N$5 renamed SD_MISO
- net N$6 renamed SD_MOSI
Changed lines of the file:
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@@
 </segment>
 </net>
-<net name="N$5" class="0">
+<net name="SD_MISO" class="0">
 <segment>
 <pinref part="IC1" gate="G$1" pin="IL4"/>
@@
 </segment>
 </net>
-<net name="N$6" class="0">
+<net name="SD_MOSI" class="0">
 <segment>
 <pinref part="IC1" gate="G$1" pin="OL3"/>
@@
 </segment>
 </net>
-<net name="N$11" class="0">
+<net name="SD_CS" class="0">
 <segment>
 <pinref part="IC1" gate="G$1" pin="OL2"/>
@@
 </segment>
 </net>
-<net name="N$15" class="0">
+<net name="SD_SCK" class="0">
 <segment>
 <pinref part="IC1" gate="G$1" pin="OL1"/>
